Commit message: Arbol de comportamiento

File: pamabot_my_world_2/urdf/turtlebot3_burger.urdf (robot description, URDF)
Before this commit: robot turtlebot3_burger, 7 links, 6 joints
Links:
- link base_link: mass 0.82573504 -> 8.2573504e-01
- link wheel_left_link: mass 0.02849894 -> 2.8498940e-02
- link wheel_right_link: mass 0.02849894 -> 2.8498940e-02

File: pamabot_my_world_2/urdf/turtlebot3_burger_pi.urdf (robot description, URDF)
Before this commit: robot turtlebot3_burger, 7 links, 6 joints
Links:
- added link camera_link; collision box size=0.015 0.030 0.027
- added link camera_rgb_frame
- added link camera_rgb_optical_frame
- link base_link: mass 0.82573504 -> 8.2573504e-01
- link wheel_left_link: mass 0.02849894 -> 2.8498940e-02
- link wheel_right_link: mass 0.02849894 -> 2.8498940e-02
Joints:
- added joint camera_joint: type fixed, parent base_link, child camera_link, origin xyz=0.063 -0.011 0.084 rpy=0 0 0
- added joint camera_rgb_joint: type fixed, parent camera_link, child camera_rgb_frame, origin xyz=0.003 0.011 0.009 rpy=0 0 0
- added joint camera_rgb_optical_joint: type fixed, parent camera_rgb_frame, child camera_rgb_optical_frame, origin xyz=0 0 0 rpy=-1.57 0 -1.57
